File: Hardware/connector_rpi/connector rpi/connector rpi.kicad_sch (KiCad schematic)
At the start: 3 parts, among them J1 Raspberry_Pi_2_3

Commit message: add
Parts:
- removed C1, C2: border_connector, pred:connector placa st7789, symbol pred:border_connector
- added J2, J3, J4, J5: Conn_01x08_Socket, symbol Connector:Conn_01x08_Socket
- added R1, R2: R0, symbol Device:R_Small
- added U1: ESP-12F, symbol ESP8266:ESP-12F
- J1: footprint Connector_PinSocket_2.54mm:PinSocket_2x20_P2.54mm_Vertical -> (none)
Connections:
- net GND: now also J2.8 (Pin_8), J3.8 (Pin_8), J4.8 (Pin_8), J5.8 (Pin_8)
- net +5V: now reaches J1.4 (5V)
- net +5V: now also J1.2 (5V), R1.1
- net SCL: now reaches J1.23 (SCLK0/GPIO11)
- net SCL: now also J2.6 (Pin_6), J3.6 (Pin_6), J4.6 (Pin_6), J5.6 (Pin_6)
- net SDA: now reaches J1.19 (MOSI0/GPIO10)
- net SDA: now also J2.5 (Pin_5), J3.5 (Pin_5), J4.5 (Pin_5), J5.5 (Pin_5)
- net DC0: now reaches J1.22 (GPIO25)
- net DC0: now also J3.3 (Pin_3)
- net CS1: now reaches J1.26 (~{CE1}/GPIO7)
- net CS1: now also J2.2 (Pin_2), J4.2 (Pin_2)
- net RES: now reaches J1.18 (GPIO24)
- net RES: now also J2.4 (Pin_4), J3.4 (Pin_4), J4.4 (Pin_4), J5.4 (Pin_4)
- net CS0: now reaches J1.24 (~{CE0}/GPIO8)
- net CS0: now also J3.2 (Pin_2), J5.2 (Pin_2)
- net +3.3V: now reaches J1.1 (3V3)
- net +3.3V: now also J1.17 (3V3), R2.1
- net RX: now reaches J1.10 (GPIO15/RXD)
- net RX: now also U1.16 (TXD)
- net BLK: now reaches J1.29 (GCLK1/GPIO5)
- net BLK: now also J2.1 (Pin_1), J3.1 (Pin_1), J4.1 (Pin_1), J5.1 (Pin_1)
- net DC1: now reaches J1.37 (GPIO26)
- net DC1: now also J2.3 (Pin_3)
- net TX: now reaches J1.8 (GPIO14/TXD)
- net TX: now also U1.15 (RXD)
- new net DC: J4.3 (Pin_3), J5.3 (Pin_3)
- new net VCC: J2.7 (Pin_7), J3.7 (Pin_7), J4.7 (Pin_7), J5.7 (Pin_7), R1.2, R2.2
Other:
- note added: "ST7789 BLK (back light) this is PWM, pull high:ON CS (chip select) DC::D/C (data command) RES (reset) if pull down TFT Reset SDA (serial data) => MOSI SCL (serial clock) => SCLK VCC GND"
